Commit message: feat(ros): ROS2 包 puppy_bringup/description/gait/worlds 与 nav_core
puppy_description(URDF xacro/控制器)、puppy_gait(gait_controller.cpp+参数+launch)、puppy_bringup(coppelia_bridge)、puppy_worlds(家庭场景 world/launch)、puppypi_adapter 驱动与状态适配；nav_core 包与 path_validator 校验脚本。

File: src/puppy_description/urdf/gazebo_control.xacro (robot description, xacro)
@@ -1,7 +1,8 @@
 <?xml version="1.0"?>
 <robot name="gazebo_control" xmlns:xacro="http://www.ros.org/wiki/xacro">
-  <xacro:macro name="gazebo_control">
+  <xacro:macro name="gazebo_control" params="use_planar_move:=true">
     <!-- 平面移动插件：直接通过 /cmd_vel 控制 base_link 速度 -->
     <!-- 最小闭环方案：先跑通 SLAM + Nav2，之后再换成足式步态 -->
+    <xacro:if value="${use_planar_move}">
     <gazebo>
       <plugin name="planar_move_controller" filename="libgazebo_ros_planar_move.so">
@@ -15,9 +16,32 @@
       </plugin>
     </gazebo>
+    </xacro:if>
+    <xacro:unless value="${use_planar_move}">
+      <ros2_control name="PuppyPiSimSystem" type="system">
+        <hardware><plugin>gazebo_ros2_control/GazeboSystem</plugin></hardware>
+        <joint name="FR_hip_yaw_joint"><command_interface name="position"/><state_interface name="position"/><state_interface name="velocity"/></joint>
+        <joint name="FR_hip_pitch_joint"><command_interface name="position"/><state_interface name="position"/><state_interface name="velocity"/></joint>
+        <joint name="FR_knee_joint"><command_interface name="position"/><state_interface name="position"/><state_interface name="velocity"/></joint>
+        <joint name="FL_hip_yaw_joint"><command_interface name="position"/><state_interface name="position"/><state_interface name="velocity"/></joint>
+        <joint name="FL_hip_pitch_joint"><command_interface name="position"/><state_interface name="position"/><state_interface name="velocity"/></joint>
+        <joint name="FL_knee_joint"><command_interface name="position"/><state_interface name="position"/><state_interface name="velocity"/></joint>
+        <joint name="RR_hip_yaw_joint"><command_interface name="position"/><state_interface name="position"/><state_interface name="velocity"/></joint>
+        <joint name="RR_hip_pitch_joint"><command_interface name="position"/><state_interface name="position"/><state_interface name="velocity"/></joint>
+        <joint name="RR_knee_joint"><command_interface name="position"/><state_interface name="position"/><state_interface name="velocity"/></joint>
+        <joint name="RL_hip_yaw_joint"><command_interface name="position"/><state_interface name="position"/><state_interface name="velocity"/></joint>
+        <joint name="RL_hip_pitch_joint"><command_interface name="position"/><state_interface name="position"/><state_interface name="velocity"/></joint>
+        <joint name="RL_knee_joint"><command_interface name="position"/><state_interface name="position"/><state_interface name="velocity"/></joint>
+      </ros2_control>
+      <gazebo>
+        <plugin filename="libgazebo_ros2_control.so" name="gazebo_ros2_control">
+          <parameters>$(find puppy_description)/config/controllers.yaml</parameters>
+        </plugin>
+      </gazebo>
+    </xacro:unless>
     <!-- Gazebo friction/dynamics for base -->
     <gazebo reference="base_link">
       <mu1>0.3</mu1>
       <mu2>0.3</mu2>
-      <gravity>false</gravity>
+      <gravity>true</gravity>
     </gazebo>
     <!-- 禁用所有腿的重力，防止机器人翻倒 -->

File: src/puppy_description/urdf/leg.xacro (robot description, xacro)
@@ -28,8 +28,10 @@
     </link>
     <!-- Hip yaw joint (fixed) -->
-    <joint name="${prefix}_hip_yaw_joint" type="fixed">
+    <joint name="${prefix}_hip_yaw_joint" type="revolute">
       <parent link="base_link"/>
       <child link="${prefix}_hip_yaw_link"/>
       <origin xyz="${x_pos} ${y_offset} 0" rpy="0 0 0"/>
+      <axis xyz="0 1 0"/>
+      <limit lower="-0.55" upper="0.55" effort="3.0" velocity="4.0"/>
     </joint>
     <!-- Hip pitch link (thigh) -->
@@ -51,8 +53,10 @@
     </link>
     <!-- Hip pitch joint (fixed) -->
-    <joint name="${prefix}_hip_pitch_joint" type="fixed">
+    <joint name="${prefix}_hip_pitch_joint" type="revolute">
       <parent link="${prefix}_hip_yaw_link"/>
       <child link="${prefix}_thigh_link"/>
       <origin xyz="0 0 0" rpy="0 0 0"/>
+      <axis xyz="0 1 0"/>
+      <limit lower="-1.35" upper="1.35" effort="3.0" velocity="5.0"/>
     </joint>
     <!-- Calf link (shin) -->
@@ -74,8 +78,10 @@
     </link>
     <!-- Knee joint (fixed) -->
-    <joint name="${prefix}_knee_joint" type="fixed">
+    <joint name="${prefix}_knee_joint" type="revolute">
       <parent link="${prefix}_thigh_link"/>
       <child link="${prefix}_calf_link"/>
       <origin xyz="0 0 ${-L1}" rpy="0 0 0"/>
+      <axis xyz="0 1 0"/>
+      <limit lower="-2.35" upper="0.15" effort="3.0" velocity="5.0"/>
     </joint>
     <!-- Foot tip (sphere for contact) -->

File: src/puppy_description/urdf/puppy.urdf.xacro (robot description, xacro)
@@ -1,4 +1,5 @@
 <?xml version="1.0"?>
 <robot name="puppy" xmlns:xacro="http://www.ros.org/wiki/xacro">
+  <xacro:arg name="use_planar_move" default="true"/>
   <!-- Include all xacro files -->
   <xacro:include filename="$(find puppy_description)/urdf/materials.xacro"/>
@@ -9,18 +10,18 @@
   <xacro:include filename="$(find puppy_description)/urdf/gazebo_control.xacro"/>
   <!-- Robot parameters -->
-  <xacro:property name="body_length" value="0.40"/>
-  <xacro:property name="body_width" value="0.22"/>
-  <xacro:property name="body_height" value="0.12"/>
-  <xacro:property name="body_mass" value="8.0"/>
-  <xacro:property name="L1" value="0.20"/>
-  <xacro:property name="L2" value="0.20"/>
-  <xacro:property name="thigh_radius" value="0.03"/>
+  <xacro:property name="body_length" value="0.30"/>
+  <xacro:property name="body_width" value="0.18"/>
+  <xacro:property name="body_height" value="0.10"/>
+  <xacro:property name="body_mass" value="2.5"/>
+  <xacro:property name="L1" value="0.105"/>
+  <xacro:property name="L2" value="0.115"/>
+  <xacro:property name="thigh_radius" value="0.022"/>
   <xacro:property name="thigh_length" value="${L1}"/>
-  <xacro:property name="calf_radius" value="0.025"/>
+  <xacro:property name="calf_radius" value="0.018"/>
   <xacro:property name="calf_length" value="${L2}"/>
-  <xacro:property name="hip_radius" value="0.04"/>
-  <xacro:property name="hip_length" value="0.06"/>
-  <xacro:property name="leg_mass" value="0.8"/>
-  <xacro:property name="stand_height" value="0.28"/>
+  <xacro:property name="hip_radius" value="0.025"/>
+  <xacro:property name="hip_length" value="0.045"/>
+  <xacro:property name="leg_mass" value="0.20"/>
+  <xacro:property name="stand_height" value="0.205"/>
   <!-- Build the robot -->
   <xacro:torso/>
@@ -33,4 +34,4 @@
   <xacro:sensors/>
   <!-- Gazebo control -->
-  <xacro:gazebo_control/>
+  <xacro:gazebo_control use_planar_move="$(arg use_planar_move)"/>
 </robot>

File: src/puppy_description/urdf/sensors.xacro (robot description, xacro)
@@ -132,7 +132,7 @@
           <ros>
             <namespace>/camera</namespace>
-            <remapping>image_raw:=rgb/image_raw</remapping>
+            <remapping>image_raw:=color/image_raw</remapping>
             <remapping>depth/image_raw:=depth/image_raw</remapping>
-            <remapping>camera_info:=rgb/camera_info</remapping>
+            <remapping>camera_info:=color/camera_info</remapping>
             <remapping>depth/camera_info:=depth/camera_info</remapping>
           </ros>
